Commit message: Doing something

File: ros2_control_demos/example_2/description/urdf/diffbot.urdf.xacro (robot description, xacro)
@@ -1,18 +1,15 @@
 <?xml version="1.0"?>
-<!-- Basic differential drive mobile base with 4 wheels -->
+<!-- Basic differential drive mobile base -->
 <robot xmlns:xacro="http://www.ros.org/wiki/xacro" name="diffdrive_robot">
   <xacro:arg name="prefix" default="" />
   <xacro:arg name="use_mock_hardware" default="false" />
   <xacro:arg name="use_sim_time" default="false" />
-  <xacro:include filename="$(find ros2_control_demo_description)/diffbot/urdf/diffbot_description_4wheels.urdf.xacro" />
+  <xacro:include filename="$(find r2m_4wd_diff_description)/r2m_4wd_diff_description/urdf/r2m_4wd_diff_description.urdf.xacro" />
   <!-- Import Rviz colors -->
-  <xacro:include filename="$(find ros2_control_demo_description)/diffbot/urdf/diffbot.materials.xacro" />
+  <!-- Materials are now referenced within the r2m_4wd_diff_description -->
   <!-- Import diffbot ros2_control description -->
-  <xacro:include filename="$(find ros2_control_demo_example_2)/ros2_control/diffbot_4wheels.ros2_control.xacro" />
-  <xacro:diffbot_4wheels prefix="$(arg prefix)" />
+  <xacro:include filename="$(find ros2_control_demo_example_2)/ros2_control/diffbot.ros2_control.xacro" />
+  <xacro:r2m_4wd_diff_description prefix="$(arg prefix)" />
   <xacro:diffbot_ros2_control
-    name="DiffBot"
-    prefix="$(arg prefix)"
-    use_mock_hardware="$(arg use_mock_hardware)"
-    use_sim_time="$(arg use_sim_time)"/>
+    name="DiffBot" prefix="$(arg prefix)" use_mock_hardware="$(arg use_mock_hardware)" use_sim_time="$(arg use_sim_time)"/>
 </robot>

File: ros2_control_demos/r2m_4wd_diff_description/r2m_4wd_diff_description/urdf/r2m_4wd_diff_description.urdf.xacro (robot description, xacro)
@@ -1,5 +1,5 @@
 <?xml version="1.0"?>
 <robot xmlns:xacro="http://www.ros.org/wiki/xacro">
-  <xacro:macro name="diffbot" params="prefix">
+  <xacro:macro name="r2m_4wd_diff_description" params="prefix">
   <!-- Constants for robot dimensions -->
   <xacro:property name="PI" value="3.1415926535897931"/>

File: submodules/ros_odrive/odrive_botwheel_explorer/description/urdf/diffbot.ros2_control.xacro (robot description, xacro)
@@ -15,17 +15,9 @@
         </hardware>
       </xacro:if>
-      <!-- Left side wheels with their respective ODrive node IDs -->
-      <joint name="${prefix}front_left_wheel_joint">
+      <joint name="${prefix}left_wheel_joint">
         <param name="node_id">0</param>
       </joint>
-      <joint name="${prefix}rear_left_wheel_joint">
+      <joint name="${prefix}right_wheel_joint">
         <param name="node_id">1</param>
-      </joint>
-      <!-- Right side wheels with their respective ODrive node IDs -->
-      <joint name="${prefix}front_right_wheel_joint">
-        <param name="node_id">2</param>
-      </joint>
-      <joint name="${prefix}rear_right_wheel_joint">
-        <param name="node_id">3</param>
       </joint>
     </ros2_control>

File: submodules/ros_odrive/odrive_botwheel_explorer/description/urdf/diffbot_description.urdf.xacro (robot description, xacro)
@@ -6,10 +6,9 @@
   <xacro:property name="base_mass" value="0.3" /> <!-- arbitrary value for base mass -->
   <xacro:property name="base_width" value="0.1" />
-  <xacro:property name="base_length" value="0.3" /> <!-- Increased length to accommodate 4 wheels -->
+  <xacro:property name="base_length" value="0.1" />
   <xacro:property name="base_height" value="0.05" />
   <xacro:property name="wheel_mass" value="0.3" /> <!-- arbitrary value for wheel mass -->
   <xacro:property name="wheel_len" value="0.020" />
   <xacro:property name="wheel_radius" value="0.015" />
-  <xacro:property name="wheel_separation_x" value="0.2" /> <!-- Separation between front and rear wheels -->
   <xacro:property name="caster_wheel_mass" value="0.1" /> <!-- arbitrary value for caster wheel mass -->
   <xacro:property name="caster_wheel_radius" value="0.015" />
@@ -20,5 +19,5 @@
       <origin xyz="0 0 0" rpy="0 0 0"/>
       <geometry>
-        <box size="${base_length} ${base_width} ${base_height}"/>
+        <box size="${base_width} ${base_length} ${base_height}"/>
       </geometry>
     </collision>
@@ -26,5 +25,5 @@
       <origin xyz="0 0 ${base_height/2}" rpy="0 0 0"/>
       <geometry>
-        <box size="${base_length} ${base_width} ${base_height}"/>
+        <box size="${base_width} ${base_length} ${base_height}"/>
       </geometry>
       <material name="orange"/>
@@ -34,19 +33,19 @@
       <mass value="${base_mass}"/>
       <inertia
-        ixx="${base_mass / 12.0 * (base_width*base_width + base_height*base_height)}" ixy="0.0" ixz="0.0"
-        iyy="${base_mass / 12.0 * (base_height*base_height + base_length*base_length)}" iyz="0.0"
-        izz="${base_mass / 12.0 * (base_length*base_length + base_width*base_width)}"/>
+        ixx="${base_mass / 12.0 * (base_length*base_length + base_height*base_height)}" ixy="0.0" ixz="0.0"
+        iyy="${base_mass / 12.0 * (base_height*base_height + base_width*base_width)}" iyz="0.0"
+        izz="${base_mass / 12.0 * (base_width*base_width + base_length*base_length)}"/>
       </inertial>
     </link>
-    <!-- Front left wheel -->
-    <joint name="${prefix}front_left_wheel_joint" type="continuous">
+    <joint name="${prefix}left_wheel_joint" type="continuous">
       <parent link="${prefix}base_link"/>
-      <child link="${prefix}front_left_wheel"/>
-      <origin xyz="${wheel_separation_x/2} -${base_width/2} ${z_offset}" rpy="0 0 0"/>
+      <child link="${prefix}left_wheel"/>
+      <origin xyz="0 -${base_width/2} ${z_offset}" rpy="0 0 0"/>
       <axis xyz="0 1 0"/>
       <dynamics damping="0.2"/>
       <limit effort="100" velocity="1.0"/>
     </joint>
-    <link name="${prefix}front_left_wheel">
+    <!-- left wheel Link -->
+    <link name="${prefix}left_wheel">
       <collision>
         <origin xyz="0 0 0" rpy="${PI/2} 0 0"/>
@@ -71,14 +70,14 @@
         </inertial>
       </link>
-    <!-- Rear left wheel -->
-    <joint name="${prefix}rear_left_wheel_joint" type="continuous">
+    <joint name="${prefix}right_wheel_joint" type="continuous">
       <parent link="${prefix}base_link"/>
-      <child link="${prefix}rear_left_wheel"/>
-      <origin xyz="${-wheel_separation_x/2} -${base_width/2} ${z_offset}" rpy="0 0 0"/>
+      <child link="${prefix}right_wheel"/>
+      <origin xyz="0 ${base_width/2} ${z_offset}" rpy="0 0 0"/>
       <axis xyz="0 1 0"/>
       <dynamics damping="0.2"/>
       <limit effort="100" velocity="1.0"/>
     </joint>
-    <link name="${prefix}rear_left_wheel">
+    <!-- right wheel Link -->
+    <link name="${prefix}right_wheel">
       <collision>
         <origin xyz="0 0 0" rpy="${PI/2} 0 0"/>
@@ -103,66 +102,60 @@
         </inertial>
       </link>
-    <!-- Front right wheel -->
-    <joint name="${prefix}front_right_wheel_joint" type="continuous">
+    <joint name="${prefix}caster_frontal_wheel_joint" type="fixed">
       <parent link="${prefix}base_link"/>
-      <child link="${prefix}front_right_wheel"/>
-      <origin xyz="${wheel_separation_x/2} ${base_width/2} ${z_offset}" rpy="0 0 0"/>
-      <axis xyz="0 1 0"/>
-      <dynamics damping="0.2"/>
-      <limit effort="100" velocity="1.0"/>
+      <child link="${prefix}caster_frontal_wheel"/>
+      <origin xyz="${base_width/2 - caster_wheel_radius} 0 ${z_offset}" rpy="0 0 0"/>
     </joint>
-    <link name="${prefix}front_right_wheel">
+    <!-- caster frontal wheel Link -->
+    <link name="${prefix}caster_frontal_wheel">
       <collision>
-        <origin xyz="0 0 0" rpy="${PI/2} 0 0"/>
+        <origin xyz="0 0 0" rpy="0 0 0"/>
         <geometry>
-          <cylinder length="${wheel_len}" radius="${wheel_radius}"/>
+          <sphere radius="${caster_wheel_radius}"/>
         </geometry>
       </collision>
       <visual>
-        <origin xyz="0 0 0" rpy="${PI/2} 0 0"/>
+        <origin xyz="0 0 0" rpy="0 0 0"/>
         <geometry>
-          <cylinder length="${wheel_len}" radius="${wheel_radius}"/>
+          <sphere radius="${caster_wheel_radius}"/>
         </geometry>
-        <material name="black"/>
+        <material name="white"/>
       </visual>
       <inertial>
-        <origin xyz="0 0 0" rpy="${PI/2} 0 0"/>
-        <mass value="${wheel_mass}"/>
+        <origin xyz="0 0 0" rpy="0 0 0"/>
+        <mass value="${caster_wheel_mass}"/>
         <inertia
-          ixx="${wheel_mass / 12.0 * (3*wheel_radius*wheel_radius + wheel_len*wheel_len)}" ixy="0.0" ixz="0.0"
-          iyy="${wheel_mass / 12.0 * (3*wheel_radius*wheel_radius + wheel_len*wheel_len)}" iyz="0.0"
-          izz="${wheel_mass / 2.0 * wheel_radius*wheel_radius}"/>
+          ixx="${caster_wheel_mass * 0.4 * (caster_wheel_radius * caster_wheel_radius)}" ixy="0.0" ixz="0.0"
+          iyy="${caster_wheel_mass * 0.4 * (caster_wheel_radius * caster_wheel_radius)}" iyz="0.0"
+          izz="${caster_wheel_mass * 0.4 * (caster_wheel_radius * caster_wheel_radius)}"/>
         </inertial>
       </link>
-    <!-- Rear right wheel -->
-    <joint name="${prefix}rear_right_wheel_joint" type="continuous">
+    <joint name="${prefix}caster_rear_wheel_joint" type="fixed">
       <parent link="${prefix}base_link"/>
-      <child link="${prefix}rear_right_wheel"/>
-      <origin xyz="${-wheel_separation_x/2} ${base_width/2} ${z_offset}" rpy="0 0 0"/>
-      <axis xyz="0 1 0"/>
-      <dynamics damping="0.2"/>
-      <limit effort="100" velocity="1.0"/>
+      <child link="${prefix}caster_rear_wheel"/>
+      <origin xyz="${-base_width/2 + caster_wheel_radius} 0 ${z_offset}" rpy="0 0 0"/>
     </joint>
-    <link name="${prefix}rear_right_wheel">
+    <!-- caster rear wheel Link -->
+    <link name="${prefix}caster_rear_wheel">
       <collision>
-        <origin xyz="0 0 0" rpy="${PI/2} 0 0"/>
+        <origin xyz="0 0 0" rpy="0 0 0"/>
         <geometry>
-          <cylinder length="${wheel_len}" radius="${wheel_radius}"/>
+          <sphere radius="${caster_wheel_radius}"/>
         </geometry>
       </collision>
       <visual>
-        <origin xyz="0 0 0" rpy="${PI/2} 0 0"/>
+        <origin xyz="0 0 0" rpy="0 0 0"/>
         <geometry>
-          <cylinder length="${wheel_len}" radius="${wheel_radius}"/>
+          <sphere radius="${caster_wheel_radius}"/>
         </geometry>
-        <material name="black"/>
+        <material name="white"/>
       </visual>
       <inertial>
-        <origin xyz="0 0 0" rpy="${PI/2} 0 0"/>
-        <mass value="${wheel_mass}"/>
+        <origin xyz="0 0 0" rpy="0 0 0"/>
+        <mass value="${caster_wheel_mass}"/>
         <inertia
-          ixx="${wheel_mass / 12.0 * (3*wheel_radius*wheel_radius + wheel_len*wheel_len)}" ixy="0.0" ixz="0.0"
-          iyy="${wheel_mass / 12.0 * (3*wheel_radius*wheel_radius + wheel_len*wheel_len)}" iyz="0.0"
-          izz="${wheel_mass / 2.0 * wheel_radius*wheel_radius}"/>
+          ixx="${caster_wheel_mass * 0.4 * (caster_wheel_radius * caster_wheel_radius)}" ixy="0.0" ixz="0.0"
+          iyy="${caster_wheel_mass * 0.4 * (caster_wheel_radius * caster_wheel_radius)}" iyz="0.0"
+          izz="${caster_wheel_mass * 0.4 * (caster_wheel_radius * caster_wheel_radius)}"/>
         </inertial>
       </link>

Commit message: Added stuff

File: ros2_control_demos/example_2/description/urdf/diffbot.urdf.xacro (robot description, xacro)
@@ -5,10 +5,10 @@
   <xacro:arg name="use_mock_hardware" default="false" />
   <xacro:arg name="use_sim_time" default="false" />
-  <xacro:include filename="$(find r2m_4wd_diff_description)/urdf/r2m_4wd_diff_description.urdf.xacro" />
+  <xacro:include filename="$(find ros2_control_demo_description)/diffbot/urdf/diffbot_description.urdf.xacro" />
   <!-- Import Rviz colors -->
-  <xacro:include filename="$(find r2m_4wd_diff_description)/urdf/diffbot.materials.xacro" />
+  <xacro:include filename="$(find ros2_control_demo_description)/diffbot/urdf/diffbot.materials.xacro" />
   <!-- Import diffbot ros2_control description -->
   <xacro:include filename="$(find ros2_control_demo_example_2)/ros2_control/diffbot.ros2_control.xacro" />
-  <xacro:r2m_4wd_diff_description prefix="$(arg prefix)" />
+  <xacro:diffbot prefix="$(arg prefix)" />
   <xacro:diffbot_ros2_control
     name="DiffBot" prefix="$(arg prefix)" use_mock_hardware="$(arg use_mock_hardware)" use_sim_time="$(arg use_sim_time)"/>

File: ros2_control_demos/ros2_control_demo_description/diffbot/urdf/diffbot_description.urdf.xacro (robot description, xacro)
@@ -1,5 +1,5 @@
 <?xml version="1.0"?>
 <robot xmlns:xacro="http://www.ros.org/wiki/xacro">
-  <xacro:macro name="r2m_4wd_diff_description" params="prefix">
+  <xacro:macro name="diffbot" params="prefix">
   <!-- Constants for robot dimensions -->
   <xacro:property name="PI" value="3.1415926535897931"/>
