Commit message: Added 4wd mod

File: ros2_control_demos/example_2/description/ros2_control/diffbot.ros2_control.xacro (robot description, xacro)
@@ -17,14 +17,28 @@
           </hardware>
         </xacro:if>
-        <joint name="${prefix}left_wheel_joint">
-          <command_interface name="velocity"/>
-          <state_interface name="position"/>
-          <state_interface name="velocity"/>
-        </joint>
-        <joint name="${prefix}right_wheel_joint">
-          <command_interface name="velocity"/>
-          <state_interface name="position"/>
-          <state_interface name="velocity"/>
-        </joint>
+        <!-- Front left wheel - ODrive 0 -->
+      <joint name="${prefix}front_left_wheel_joint">
+        <command_interface name="velocity"/>
+        <state_interface name="position"/>
+        <state_interface name="velocity"/>
+      </joint>
+      <!-- Front right wheel - ODrive 1 -->
+      <joint name="${prefix}front_right_wheel_joint">
+        <command_interface name="velocity"/>
+        <state_interface name="position"/>
+        <state_interface name="velocity"/>
+      </joint>
+      <!-- Rear left wheel - ODrive 2 -->
+      <joint name="${prefix}rear_left_wheel_joint">
+        <command_interface name="velocity"/>
+        <state_interface name="position"/>
+        <state_interface name="velocity"/>
+      </joint>
+      <!-- Rear right wheel - ODrive 3 -->
+      <joint name="${prefix}rear_right_wheel_joint">
+        <command_interface name="velocity"/>
+        <state_interface name="position"/>
+        <state_interface name="velocity"/>
+      </joint>
      </ros2_control>
     </xacro:if>
@@ -35,16 +49,32 @@
           <param name="can">can0</param>
         </hardware>
-        <joint name="${prefix}left_wheel_joint">
-          <param name="node_id">0</param>
-          <command_interface name="velocity"/>
-          <state_interface name="position"/>
-          <state_interface name="velocity"/>
-        </joint>
-        <joint name="${prefix}right_wheel_joint">
-          <param name="node_id">1</param>
-          <command_interface name="velocity"/>
-          <state_interface name="position"/>
-          <state_interface name="velocity"/>
-        </joint>
+        <!-- Front left wheel - ODrive 0 -->
+      <joint name="${prefix}front_left_wheel_joint">
+        <param name="node_id">0</param>
+        <command_interface name="velocity"/>
+        <state_interface name="position"/>
+        <state_interface name="velocity"/>
+      </joint>
+      <!-- Front right wheel - ODrive 1 -->
+      <joint name="${prefix}front_right_wheel_joint">
+        <param name="node_id">1</param>
+        <command_interface name="velocity"/>
+        <state_interface name="position"/>
+        <state_interface name="velocity"/>
+      </joint>
+      <!-- Rear left wheel - ODrive 2 -->
+      <joint name="${prefix}rear_left_wheel_joint">
+        <param name="node_id">2</param>
+        <command_interface name="velocity"/>
+        <state_interface name="position"/>
+        <state_interface name="velocity"/>
+      </joint>
+      <!-- Rear right wheel - ODrive 3 -->
+      <joint name="${prefix}rear_right_wheel_joint">
+        <param name="node_id">3</param>
+        <command_interface name="velocity"/>
+        <state_interface name="position"/>
+        <state_interface name="velocity"/>
+      </joint>
       </ros2_control>
    </xacro:unless>

File: ros2_control_demos/example_2/ros2_control/diffbot.ros2_control.xacro (robot description, xacro)
@@ -15,17 +15,31 @@
         </hardware>
       </xacro:if>
-      <!-- Left side wheels controlled by motor driver 0 -->
+      <!-- Front left wheel - ODrive 0 -->
       <joint name="${prefix}front_left_wheel_joint">
         <param name="node_id">0</param>
+        <command_interface name="velocity"/>
+        <state_interface name="position"/>
+        <state_interface name="velocity"/>
       </joint>
-      <joint name="${prefix}rear_left_wheel_joint">
-        <param name="node_id">0</param>
-      </joint>
-      <!-- Right side wheels controlled by motor driver 1 -->
+      <!-- Front right wheel - ODrive 1 -->
       <joint name="${prefix}front_right_wheel_joint">
         <param name="node_id">1</param>
+        <command_interface name="velocity"/>
+        <state_interface name="position"/>
+        <state_interface name="velocity"/>
       </joint>
+      <!-- Rear left wheel - ODrive 2 -->
+      <joint name="${prefix}rear_left_wheel_joint">
+        <param name="node_id">2</param>
+        <command_interface name="velocity"/>
+        <state_interface name="position"/>
+        <state_interface name="velocity"/>
+      </joint>
+      <!-- Rear right wheel - ODrive 3 -->
       <joint name="${prefix}rear_right_wheel_joint">
-        <param name="node_id">1</param>
+        <param name="node_id">3</param>
+        <command_interface name="velocity"/>
+        <state_interface name="position"/>
+        <state_interface name="velocity"/>
       </joint>
     </ros2_control>

File: ros2_control_demos/ros2_control_demo_description/diffbot/urdf/diffbot_description.urdf.xacro (robot description, xacro)
@@ -4,13 +4,12 @@
   <!-- Constants for robot dimensions -->
   <xacro:property name="PI" value="3.1415926535897931"/>
-  <xacro:property name="base_mass" value="0.3" /> <!-- arbitrary value for base mass -->
-  <xacro:property name="base_width" value="0.1" />
-  <xacro:property name="base_length" value="0.1" />
-  <xacro:property name="base_height" value="0.05" />
+  <xacro:property name="base_mass" value="1.0" /> <!-- increased value for base mass -->
+  <xacro:property name="base_width" value="0.6" /> <!-- modified to 0.6 meters width -->
+  <xacro:property name="base_length" value="1.1" /> <!-- modified to 1.1 meters length -->
+  <xacro:property name="base_height" value="0.1" /> <!-- increased height -->
   <xacro:property name="wheel_mass" value="0.3" /> <!-- arbitrary value for wheel mass -->
-  <xacro:property name="wheel_len" value="0.020" />
-  <xacro:property name="wheel_radius" value="0.015" />
-  <xacro:property name="caster_wheel_mass" value="0.1" /> <!-- arbitrary value for caster wheel mass -->
-  <xacro:property name="caster_wheel_radius" value="0.015" />
+  <xacro:property name="wheel_len" value="0.050" /> <!-- increased wheel length -->
+  <xacro:property name="wheel_radius" value="0.075" /> <!-- increased wheel radius -->
+  <xacro:property name="wheel_axle_distance" value="0.8" /> <!-- distance between front and rear axles -->
   <xacro:property name="z_offset" value="-${base_height/2}" /> <!-- Space btw top of beam and the each joint -->
   <!-- Base Link -->
@@ -19,5 +18,5 @@
       <origin xyz="0 0 0" rpy="0 0 0"/>
       <geometry>
-        <box size="${base_width} ${base_length} ${base_height}"/>
+        <box size="${base_length} ${base_width} ${base_height}"/>
       </geometry>
     </collision>
@@ -25,5 +24,5 @@
       <origin xyz="0 0 ${base_height/2}" rpy="0 0 0"/>
       <geometry>
-        <box size="${base_width} ${base_length} ${base_height}"/>
+        <box size="${base_length} ${base_width} ${base_height}"/>
       </geometry>
       <material name="orange"/>
@@ -33,19 +32,20 @@
       <mass value="${base_mass}"/>
       <inertia
-        ixx="${base_mass / 12.0 * (base_length*base_length + base_height*base_height)}" ixy="0.0" ixz="0.0"
-        iyy="${base_mass / 12.0 * (base_height*base_height + base_width*base_width)}" iyz="0.0"
-        izz="${base_mass / 12.0 * (base_width*base_width + base_length*base_length)}"/>
+        ixx="${base_mass / 12.0 * (base_width*base_width + base_height*base_height)}" ixy="0.0" ixz="0.0"
+        iyy="${base_mass / 12.0 * (base_length*base_length + base_height*base_height)}" iyz="0.0"
+        izz="${base_mass / 12.0 * (base_length*base_length + base_width*base_width)}"/>
       </inertial>
     </link>
-    <joint name="${prefix}left_wheel_joint" type="continuous">
+    <!-- Front Left Wheel Joint -->
+    <joint name="${prefix}front_left_wheel_joint" type="continuous">
       <parent link="${prefix}base_link"/>
-      <child link="${prefix}left_wheel"/>
-      <origin xyz="0 -${base_width/2} ${z_offset}" rpy="0 0 0"/>
+      <child link="${prefix}front_left_wheel"/>
+      <origin xyz="${wheel_axle_distance/2} -${base_width/2} ${z_offset}" rpy="0 0 0"/>
       <axis xyz="0 1 0"/>
       <dynamics damping="0.2"/>
       <limit effort="100" velocity="1.0"/>
     </joint>
-    <!-- left wheel Link -->
-    <link name="${prefix}left_wheel">
+    <!-- Front Left Wheel Link -->
+    <link name="${prefix}front_left_wheel">
       <collision>
         <origin xyz="0 0 0" rpy="${PI/2} 0 0"/>
@@ -70,14 +70,15 @@
         </inertial>
       </link>
-    <joint name="${prefix}right_wheel_joint" type="continuous">
+    <!-- Front Right Wheel Joint -->
+    <joint name="${prefix}front_right_wheel_joint" type="continuous">
       <parent link="${prefix}base_link"/>
-      <child link="${prefix}right_wheel"/>
-      <origin xyz="0 ${base_width/2} ${z_offset}" rpy="0 0 0"/>
+      <child link="${prefix}front_right_wheel"/>
+      <origin xyz="${wheel_axle_distance/2} ${base_width/2} ${z_offset}" rpy="0 0 0"/>
       <axis xyz="0 1 0"/>
       <dynamics damping="0.2"/>
       <limit effort="100" velocity="1.0"/>
     </joint>
-    <!-- right wheel Link -->
-    <link name="${prefix}right_wheel">
+    <!-- Front Right Wheel Link -->
+    <link name="${prefix}front_right_wheel">
       <collision>
         <origin xyz="0 0 0" rpy="${PI/2} 0 0"/>
@@ -102,60 +103,68 @@
         </inertial>
       </link>
-    <joint name="${prefix}caster_frontal_wheel_joint" type="fixed">
+    <!-- Rear Left Wheel Joint -->
+    <joint name="${prefix}rear_left_wheel_joint" type="continuous">
       <parent link="${prefix}base_link"/>
-      <child link="${prefix}caster_frontal_wheel"/>
-      <origin xyz="${base_width/2 - caster_wheel_radius} 0 ${z_offset}" rpy="0 0 0"/>
+      <child link="${prefix}rear_left_wheel"/>
+      <origin xyz="${-wheel_axle_distance/2} -${base_width/2} ${z_offset}" rpy="0 0 0"/>
+      <axis xyz="0 1 0"/>
+      <dynamics damping="0.2"/>
+      <limit effort="100" velocity="1.0"/>
     </joint>
-    <!-- caster frontal wheel Link -->
-    <link name="${prefix}caster_frontal_wheel">
+    <!-- Rear Left Wheel Link -->
+    <link name="${prefix}rear_left_wheel">
       <collision>
-        <origin xyz="0 0 0" rpy="0 0 0"/>
+        <origin xyz="0 0 0" rpy="${PI/2} 0 0"/>
         <geometry>
-          <sphere radius="${caster_wheel_radius}"/>
+          <cylinder length="${wheel_len}" radius="${wheel_radius}"/>
         </geometry>
       </collision>
       <visual>
-        <origin xyz="0 0 0" rpy="0 0 0"/>
+        <origin xyz="0 0 0" rpy="${PI/2} 0 0"/>
         <geometry>
-          <sphere radius="${caster_wheel_radius}"/>
+          <cylinder length="${wheel_len}" radius="${wheel_radius}"/>
         </geometry>
-        <material name="white"/>
+        <material name="black"/>
       </visual>
       <inertial>
-        <origin xyz="0 0 0" rpy="0 0 0"/>
-        <mass value="${caster_wheel_mass}"/>
+        <origin xyz="0 0 0" rpy="${PI/2} 0 0"/>
+        <mass value="${wheel_mass}"/>
         <inertia
-          ixx="${caster_wheel_mass * 0.4 * (caster_wheel_radius * caster_wheel_radius)}" ixy="0.0" ixz="0.0"
-          iyy="${caster_wheel_mass * 0.4 * (caster_wheel_radius * caster_wheel_radius)}" iyz="0.0"
-          izz="${caster_wheel_mass * 0.4 * (caster_wheel_radius * caster_wheel_radius)}"/>
+          ixx="${wheel_mass / 12.0 * (3*wheel_radius*wheel_radius + wheel_len*wheel_len)}" ixy="0.0" ixz="0.0"
+          iyy="${wheel_mass / 12.0 * (3*wheel_radius*wheel_radius + wheel_len*wheel_len)}" iyz="0.0"
+          izz="${wheel_mass / 2.0 * wheel_radius*wheel_radius}"/>
         </inertial>
       </link>
-    <joint name="${prefix}caster_rear_wheel_joint" type="fixed">
+    <!-- Rear Right Wheel Joint -->
+    <joint name="${prefix}rear_right_wheel_joint" type="continuous">
       <parent link="${prefix}base_link"/>
-      <child link="${prefix}caster_rear_wheel"/>
-      <origin xyz="${-base_width/2 + caster_wheel_radius} 0 ${z_offset}" rpy="0 0 0"/>
+      <child link="${prefix}rear_right_wheel"/>
+      <origin xyz="${-wheel_axle_distance/2} ${base_width/2} ${z_offset}" rpy="0 0 0"/>
+      <axis xyz="0 1 0"/>
+      <dynamics damping="0.2"/>
+      <limit effort="100" velocity="1.0"/>
     </joint>
-    <!-- caster rear wheel Link -->
-    <link name="${prefix}caster_rear_wheel">
+    <!-- Rear Right Wheel Link -->
+    <link name="${prefix}rear_right_wheel">
       <collision>
-        <origin xyz="0 0 0" rpy="0 0 0"/>
+        <origin xyz="0 0 0" rpy="${PI/2} 0 0"/>
         <geometry>
-          <sphere radius="${caster_wheel_radius}"/>
+          <cylinder length="${wheel_len}" radius="${wheel_radius}"/>
         </geometry>
       </collision>
       <visual>
-        <origin xyz="0 0 0" rpy="0 0 0"/>
+        <origin xyz="0 0 0" rpy="${PI/2} 0 0"/>
         <geometry>
-          <sphere radius="${caster_wheel_radius}"/>
+          <cylinder length="${wheel_len}" radius="${wheel_radius}"/>
         </geometry>
-        <material name="white"/>
+        <material name="black"/>
       </visual>
       <inertial>
-        <origin xyz="0 0 0" rpy="0 0 0"/>
-        <mass value="${caster_wheel_mass}"/>
+        <origin xyz="0 0 0" rpy="${PI/2} 0 0"/>
+        <mass value="${wheel_mass}"/>
         <inertia
-          ixx="${caster_wheel_mass * 0.4 * (caster_wheel_radius * caster_wheel_radius)}" ixy="0.0" ixz="0.0"
-          iyy="${caster_wheel_mass * 0.4 * (caster_wheel_radius * caster_wheel_radius)}" iyz="0.0"
-          izz="${caster_wheel_mass * 0.4 * (caster_wheel_radius * caster_wheel_radius)}"/>
+          ixx="${wheel_mass / 12.0 * (3*wheel_radius*wheel_radius + wheel_len*wheel_len)}" ixy="0.0" ixz="0.0"
+          iyy="${wheel_mass / 12.0 * (3*wheel_radius*wheel_radius + wheel_len*wheel_len)}" iyz="0.0"
+          izz="${wheel_mass / 2.0 * wheel_radius*wheel_radius}"/>
         </inertial>
       </link>
